File: BlockBox.brd (EAGLE design)
At the start: 123.2 x 119.4 mm, 344 parts, among them J100 TE-770966, J400 ICSP, J401 ZX62D-B-5PA8, J402 AUX, J403 LED, J404 SWLED, J405 USB1, J406 USB2, Q100 TK3R1E04PL, Q101 TK3R1E04PL, Q102 IPP052N06L3 G, Q103 IPP052N06L3 G, Q104 IPP052N06L3 G, Q105 IPP052N06L3 G, Q106 TK3R1E04PL, Q200 IRFB4510PBF, Q201 IRFB4510PBF, Q202 BUK9Y43-60E, Q203 DMP4065S, Q300 NMOS, Q400 NMOS, Q401 NMOS, Q402 NMOS, Q403 DMG2302UK, Q404 DMG2302UK, Q405 DMG2302UK, Q406 NMOS, Q407 NMOS, SW100 PWRSW, SW400 DIPSW-SPDT-5, SW401 MFB, SW402 BTN1, SW403 BTN2, SW404 BTN3, SW405 BTN4, SW406 BTN5, SW407 RESET, SW408 LCDBL, U100 BQ77915, U101 MAX1737, U102 LM74700-Q1, U103 LM74700-Q1, U104 LM74700-Q1, U200 LM5022, U201 LM3488, U202 LM25085, U203 LDO-3.3V, U204 LDO-3.8V, U300 TPA3255, U301 NCS20071, U302 LM2902, U303 LM2902, U304 LM2902, U305 LM2904, U306 NCS20071, U400 PIC18LF4_K42, U401 FT230XS, U402 NCS20071

Commit message: Final checks and fixes applied.
Parts:
- moved FAN300 1.27 mm to (79.6, 116.0)
- moved RT300 1.27 mm to (82.2, 116.0)
Routing:
- net AMP_FAN_-: track 18.7 -> 20.0 mm
- net AMP_FAN_+: track 24.2 -> 25.5 mm
- net AMP_FAN_SENSE: track 30.1 -> 31.4 mm
- net 12V: track 234.4 -> 235.7 mm
- net GND: vias 150 -> 148
Changed lines of the file:
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@@
 </layers>
 <board>
-<fusionsync huburn="a.cGVyc29uYWw6dWUyYmY1N2E4" projecturn="a.cGVyc29uYWw6dWUyYmY1N2E4IzIwMTkwODEwMjA3OTY0MjA2" f3durn="urn:adsk.wipprod:dm.lineage:C4QzSxdCRISNVdHAh5Jr5w" pcbguid="86e9383b-d561-4bab-9b8a-9f133792bf8a" lastpulledtime="" lastsyncedchangeguid="05967af9-933a-3850-478c-5109f884f13f"/>
+<fusionsync huburn="a.cGVyc29uYWw6dWUyYmY1N2E4" projecturn="a.cGVyc29uYWw6dWUyYmY1N2E4IzIwMTkwODEwMjA3OTY0MjA2" f3durn="urn:adsk.wipprod:dm.lineage:C4QzSxdCRISNVdHAh5Jr5w" pcbguid="86e9383b-d561-4bab-9b8a-9f133792bf8a" lastpulledtime="" lastsyncedchangeguid="5e5af9f3-0308-b943-c9c9-4bffa0fe9f98"/>
 <plain>
 <wire x1="121.92" y1="119.38" x2="1.27" y2="119.38" width="0" layer="20"/>
@@
 <wire x1="123.19" y1="1.27" x2="123.19" y2="118.11" width="0" layer="20"/>
 <wire x1="123.19" y1="118.11" x2="121.92" y2="119.38" width="0" layer="20" curve="90"/>
-<text x="76.581" y="117.983" size="1.27" layer="21" font="vector" ratio="12" rot="R90">+</text>
+<text x="77.851" y="117.983" size="1.27" layer="21" font="vector" ratio="12" rot="R90">+</text>
 <wire x1="27.178" y1="29.21" x2="18.5928" y2="29.21" width="1.778" layer="29"/>
 <wire x1="18.5928" y1="29.21" x2="17.9578" y2="29.845" width="1.778" layer="29"/>
@@
 <attribute name="VALUE" x="106.68" y="85.09" size="1.27" layer="27" font="vector" ratio="12"/>
 </element>
-<element name="FAN300" library="BW-PassiveMechanical" package="WIRE-2P-SIMPLE" value="12V &lt;50mA" x="78.359" y="115.951" smashed="yes" rot="R270">
-<attribute name="NAME" x="76.708" y="111.252" size="1.27" layer="25" font="vector" ratio="12" rot="R90"/>
+<element name="FAN300" library="BW-PassiveMechanical" package="WIRE-2P-SIMPLE" value="12V &lt;50mA" x="79.629" y="115.951" smashed="yes" rot="R270">
+<attribute name="NAME" x="77.978" y="111.252" size="1.27" layer="25" font="vector" ratio="12" rot="R90"/>
 </element>
 <element name="H300" library="BW-PassiveMechanical" package="ATS-CPX030030030-173-C2-R0" override_package3d_urn="urn:adsk.eagle:package:12552342/2" override_package_urn="urn:adsk.eagle:footprint:12552343/1" value="ATS-CPX030030030-173-C2-R0" x="54.61" y="96.52" smashed="yes">
@@
 <element name="Q100" library="BW-Active" package="TO220BV" value="TK3R1E04PL" x="35.814" y="12.192" smashed="yes">
 <attribute name="NAME" x="31.496" y="6.5278" size="1.016" layer="25" font="vector" ratio="15"/>
-<attribute name="VALUE" x="31.496" y="2.667" size="1.016" layer="27" font="vector" ratio="15"/>
+<attribute name="VALUE" x="30.48" y="2.667" size="1.016" layer="27" font="vector" ratio="15"/>
 </element>
 <element name="Q101" library="BW-Active" package="TO220BV" value="TK3R1E04PL" x="35.814" y="23.622" smashed="yes">
@@
 </element>
 <element name="R206" library="resistor" library_urn="urn:adsk.eagle:library:348" package="R1206" package3d_urn="urn:adsk.eagle:package:23540/2" value="8mΩ" x="120.65" y="59.817" smashed="yes" rot="R270">
-<attribute name="NAME" x="116.078" y="64.008" size="1.27" layer="25" font="vector" ratio="12"/>
-<attribute name="VALUE" x="116.459" y="62.611" size="1.27" layer="27" font="vector" ratio="12"/>
+<attribute name="NAME" x="115.697" y="64.008" size="1.27" layer="25" font="vector" ratio="12"/>
+<attribute name="VALUE" x="116.078" y="62.484" size="1.27" layer="27" font="vector" ratio="12"/>
 </element>
 <element name="R207" library="resistor" library_urn="urn:adsk.eagle:library:348" package="R0603" package3d_urn="urn:adsk.eagle:package:23555/3" value="23.2kΩ" x="92.202" y="51.308" smashed="yes" rot="MR90">
@@
 <attribute name="VALUE" x="44.831" y="60.706" size="1.016" layer="28" font="vector" ratio="15" rot="MR0"/>
 </element>
-<element name="RT300" library="BW-PassiveMechanical" package="WIRE-2P-SIMPLE" value="103AT" x="80.899" y="115.951" smashed="yes" rot="R270">
-<attribute name="NAME" x="83.693" y="113.411" size="1.27" layer="25" font="vector" ratio="12" rot="R90"/>
-<attribute name="VALUE" x="85.344" y="113.411" size="1.27" layer="27" font="vector" ratio="12" rot="R90"/>
+<element name="RT300" library="BW-PassiveMechanical" package="WIRE-2P-SIMPLE" value="103AT" x="82.169" y="115.951" smashed="yes" rot="R270">
+<attribute name="NAME" x="84.963" y="113.411" size="1.27" layer="25" font="vector" ratio="12" rot="R90"/>
+<attribute name="VALUE" x="86.614" y="113.411" size="1.27" layer="27" font="vector" ratio="12" rot="R90"/>
 </element>
 <element name="RV300" library="BW-PassiveMechanical" package="TC33X-2" value="20kΩ" x="32.131" y="115.824" smashed="yes" rot="R90">
@@
 <via x="120.65" y="61.214" extent="1-16" drill="0.3"/>
 <via x="117.856" y="60.833" extent="1-16" drill="0.3"/>
-<via x="118.237" y="61.849" extent="1-16" drill="0.3"/>
-<via x="118.745" y="62.738" extent="1-16" drill="0.3"/>
-<via x="119.507" y="63.5" extent="1-16" drill="0.3"/>
-<via x="120.523" y="64.008" extent="1-16" drill="0.3"/>
-<via x="121.666" y="64.135" extent="1-16" drill="0.3"/>
+<via x="118.364" y="62.611" extent="1-16" drill="0.3"/>
+<via x="119.761" y="63.754" extent="1-16" drill="0.3"/>
+<via x="121.539" y="64.135" extent="1-16" drill="0.3"/>
 <via x="77.47" y="57.15" extent="1-16" drill="0.3"/>
 <via x="78.74" y="57.15" extent="1-16" drill="0.3"/>
@@
 <wire x1="58.363" y1="117.322" x2="58.521" y2="117.322" width="0.1524" layer="16"/>
 <wire x1="58.521" y1="117.322" x2="59.5376" y2="118.3386" width="0.1524" layer="16"/>
-<wire x1="59.5376" y1="118.3386" x2="79.7814" y2="118.3386" width="0.1524" layer="16"/>
-<wire x1="79.7814" y1="118.3386" x2="80.899" y2="117.221" width="0.1524" layer="16"/>
+<wire x1="59.5376" y1="118.3386" x2="81.0514" y2="118.3386" width="0.1524" layer="16"/>
+<wire x1="81.0514" y1="118.3386" x2="82.169" y2="117.221" width="0.1524" layer="16"/>
 <wire x1="48.199" y1="104.521" x2="48.199" y2="115.5852" width="0.1524" layer="16"/>
 <wire x1="58.2174" y1="117.322" x2="58.363" y2="117.322" width="0.1524" layer="16"/>
@@
 <wire x1="60.763" y1="117.322" x2="60.931125" y2="117.322" width="0.1524" layer="16"/>
 <wire x1="60.931125" y1="117.322" x2="61.541325" y2="117.9322" width="0.1524" layer="16"/>
-<wire x1="77.6478" y1="117.9322" x2="78.359" y2="117.221" width="0.1524" layer="16"/>
-<wire x1="61.541325" y1="117.9322" x2="77.6478" y2="117.9322" width="0.1524" layer="16"/>
+<wire x1="78.9178" y1="117.9322" x2="79.629" y2="117.221" width="0.1524" layer="16"/>
+<wire x1="61.541325" y1="117.9322" x2="78.9178" y2="117.9322" width="0.1524" layer="16"/>
 <wire x1="55.372" y1="117.182" x2="55.411" y2="117.182" width="0.1524" layer="16"/>
 <wire x1="59.7402" y1="117.322" x2="60.763" y2="117.322" width="0.1524" layer="16"/>
@@
 <contactref element="FAN300" pad="2"/>
 <wire x1="62.695" y1="112.268" x2="62.8904" y2="112.268" width="0.1524" layer="16"/>
-<wire x1="76.5556" y1="114.681" x2="78.359" y2="114.681" width="0.1524" layer="16"/>
+<wire x1="76.5556" y1="114.681" x2="79.629" y2="114.681" width="0.1524" layer="16"/>
 <wire x1="62.8904" y1="112.268" x2="67.7418" y2="117.1194" width="0.1524" layer="16"/>
 <wire x1="67.7418" y1="117.1194" x2="74.1172" y2="117.1194" width="0.1524" layer="16"/>
@@
 <wire x1="60.763" y1="115.342" x2="65.3914625" y2="115.342" width="0.1524" layer="16"/>
 <wire x1="67.5752625" y1="117.5258" x2="74.5123375" y2="117.5258" width="0.1524" layer="16"/>
-<wire x1="79.629" y1="115.951" x2="80.899" y2="114.681" width="0.1524" layer="16"/>
+<wire x1="80.899" y1="115.951" x2="82.169" y2="114.681" width="0.1524" layer="16"/>
 <wire x1="65.3914625" y1="115.342" x2="67.5752625" y2="117.5258" width="0.1524" layer="16"/>
 <wire x1="74.5123375" y1="117.5258" x2="76.0871375" y2="115.951" width="0.1524" layer="16"/>
-<wire x1="76.0871375" y1="115.951" x2="79.629" y2="115.951" width="0.1524" layer="16"/>
+<wire x1="76.0871375" y1="115.951" x2="80.899" y2="115.951" width="0.1524" layer="16"/>
 </signal>
 <signal name="AMP_FAN_GATE">
