File: BlockBox.sch (EAGLE design)
At the start: 268 parts, among them J100 PWRSW, Q100 TK3R1E04PL, Q101 TK3R1E04PL, Q102 IPP052N06L3 G, Q103 IPP052N06L3 G, Q104 IPP052N06L3 G, Q105 IPP052N06L3 G, Q106 TK3R1E04PL, Q200 IRFB4510PBF, Q201 IRFB4510PBF, Q202 BUK9Y43-60E, Q203 DMP4065S-7, Q300 NMOS, U100 BQ77915, U101 MAX1737, U102 LM74700-Q1, U103 LM74700-Q1, U104 LM74700-Q1, U200 LM5022, U201 LM3488, U202 LM25085, U203 MIC5504-3.3YM5-TR, U204 MIC5205-3.8YM5-TR, U300 TPA3255, U301 NCS20071, U302 LM2902, U303 LM2902, U304 LM2902, U305 NCS20071

Commit message: Schematic mostly done, added Multisim circuit files
Parts:
- removed U305: NCS20071, BW-Active:NCS20071
- added C356, C357: 10µF, rcl:C-EUC0805
- added C358: 2.2µF, rcl:C-EUC0603
- added C400, C401, C402: 0.1µF, rcl:C-EUC0805
- added C403, C404, C405, C406, C407: 15pF, rcl:C-EUC0603
- added D103: (no value), BW-Active:DO-219AB-ZENER
- added D400: D5V0L2B3SO, BW-Active:SOT23-TVS
- added DN300: MD_S, BW-Active:MD_S
- added F100: 15A, BW-PassiveMechanical:2410-FUSE
- added J400: PINHD-1X8, BW-Connectors:PINHD-1X8
- added J401: ZX62D-B-5PA8, BW-Connectors:ZX62D-B-5PA8
- added J402: AUX, BW-Connectors:GEN-3PIN
- added J403: LED, BW-Connectors:GEN-4PIN
- added Q400, Q401, Q402: NMOS, BW-Active:SOT23-N-MOSFET
- added Q403, Q404, Q405: DMG2302UK, BW-Active:SOT23-N-MOSFET
- added R341, R343, R344, R346, R348, R401, R402, R403, R404, R405: 10kΩ, resistor:R-US_R0805
- added R342: 1kΩ, resistor:R-US_R0805
- added R345, R347: 20kΩ, resistor:R-US_R0603
- added R400: 330Ω, resistor:R-US_R0805
- added RV303: 20kΩ, BW-PassiveMechanical:TC33X-2
- added RV400: 10kΩ, BW-PassiveMechanical:TC33X-2
- added SJ400: 3.3V-5V, jumper:SJ2W
- added SJ401: ADAP, jumper:SJ
- added SJ402: VBUS, jumper:SJ
- added SJ403: FTRESET, jumper:SJ
- added SW100: PWRSW, BW-PassiveMechanical:WIRED-SWITCH-NO
- added SW400: DIPSW-SPDT-5, BW-PassiveMechanical:DIPSW-SPDT-5
- added SW401: MFB, BW-PassiveMechanical:WIRED-SWITCH-NO
- added SW402: BTN1, BW-PassiveMechanical:WIRED-SWITCH-NO
- added SW403: BTN2, BW-PassiveMechanical:WIRED-SWITCH-NO
- added SW404: BTN3, BW-PassiveMechanical:WIRED-SWITCH-NO
- added SW405: BTN4, BW-PassiveMechanical:WIRED-SWITCH-NO
- added SW406: BTN5, BW-PassiveMechanical:WIRED-SWITCH-NO
- added SW407: RESET, BW-PassiveMechanical:WIRED-SWITCH-NO
- added SW408: LCD_BL, BW-PassiveMechanical:WIRED-SWITCH-NO
- added SW409: LEDSW, BW-PassiveMechanical:WIRED-SWITCH-NO
- added U400: PIC18LF4_K42-I/PT, BW-Active:PIC18LF4_K42-I/PT
- added U401: FT230XS, ftdichip:FT230XS
- added U405: LM2904, BW-Active:LM2904
- added U406: NCS20071, BW-Active:NCS20071
- added XDS400: HD44780_LCD-CON, BW-Active:HD44780_LCD-CON
- J100: value PWRSW -> TE-770966; device BW-Connectors:GEN-2PIN -> BW-Connectors:TE-770966
Connections:
- net !CHG_SHDN renamed CHG_!SHDN
- removed net !CHG_FASTCHG: U101.!FASTCHG
- removed net !CHG_FAULT: U101.!FAULT
- removed net !CHG_FULLCHG: U101.!FULLCHG
- new net BM_!RST: A400.!RST, U400.RB4
- new net BM_ADAP_IN: A400.ADAP_IN, SJ401.2
- new net BM_AIL: A400.AIL, D400.2, J402A.P$1
- new net BM_AIR: A400.AIR, D400.1, J402B.P$1
- new net BM_EAN: A400.EAN, SW400D.P
- new net BM_HCI_RXD: A400.HCI_RXD, SW400A.P
- new net BM_HCI_TXD: A400.HCI_TXD, SW400B.P
- new net BM_LED1: A400.LED1, U400.RB2
- new net BM_LED2: A400.LED2, U400.RB3
- new net BM_MFB: A400.MFB, SW401.1
- new net BM_MIC_N: A400.MIC1_N, R403.2
- new net BM_MIC_P: A400.MIC1_P, R402.2
- new net BM_P0_1: A400.P0_1, C406.1, SW405.1
- new net BM_P0_2: A400.P0_2, C403.1, SW402.1
- new net BM_P0_3: A400.P0_3, C407.1, SW406.1
- new net BM_P0_5: A400.P0_5, C405.1, SW404.1
- new net BM_P1_5: A400.P1_5, Q402.G
- new net BM_P2_0: A400.P2_0, SW400C.P
- new net BM_P2_4: A400.P2_4, SW400E.P
- new net BM_P2_7: A400.P2_7, C404.1, SW403.1
- new net BM_SYS_PWR: A400.SYS_PWR, SW401.2
- new net CHG_!FASTCHG: U101.!FASTCHG, U400.RD0
- new net CHG_!FAULT: U101.!FAULT, U400.RD2
- new net CHG_!FULLCHG: U101.!FULLCHG, U400.RD1
- new net FT_!CTS: R405.2, U401.!CTS
- new net FT_!RESET: SJ403.2, U401.!RESET
- new net FT_RXD: SW400B.S, U401.RXD
- new net FT_TXD: SW400A.S, U401.TXD
- new net LCD_!E: U400.RE2, XDS400.!E
- new net LCD_A: SJ400.2, XDS400.A
- new net LCD_BL_EN: Q400.G, U400.RC0
- new net LCD_D0: U400.RA0, XDS400.D0
- new net LCD_D1: U400.RA1, XDS400.D1
- new net LCD_D2: U400.RA2, XDS400.D2
- new net LCD_D3: U400.RA3, XDS400.D3
- new net LCD_D4: U400.RA4, XDS400.D4
- new net LCD_D6: U400.RA6, XDS400.D6
- new net LCD_D7: U400.RA7, XDS400.D7
- new net LCD_K: Q400.D, XDS400.K
- new net LCD_RS: U400.RE0, XDS400.RS
- new net LCD_RW: U400.RE1, XDS400.RW
- new net LCD_V0: RV400.S, XDS400.V0
- new net LDC_D5: U400.RA5, XDS400.D5
- new net LED_B: J403D.P$1, Q405.D
- new net LED_G: J403B.P$1, Q404.D
- new net LED_R: J403C.P$1, Q403.D
- new net MCU_!MCLR: J400.1, R400.2, U400.VPP/!MCLR!/RE3
- new net MCU_!MCLR!_FILTERED: C402.1, R400.1, R401.1, SW407.2
- new net MCU_AMP_RESET: Q401.G, U400.RC4
- new net MCU_BL_SW: SW408.1, U400.RC1
- new net MCU_ICSPCLK: J400.5, U400.ICSPCLK/RB6
- new net MCU_ICSPDAT: J400.4, U400.ICSPDAT/RB7
- new net MCU_LED_B: Q405.G, U400.RD6
- new net MCU_LED_G: Q404.G, U400.RD5
- new net MCU_LED_R: Q403.G, U400.RD4
- new net MCU_LED_SW: SW409.1, U400.RC6
- new net MCU_UART_RX: SW400B.O, U400.RB1
- new net MCU_UART_TX: SW400A.O, U400.RB0
- new net N$1: J401.D+, U401.USBDP
- new net N$2: J401.D-, U401.USBDM
- new net N$3: J401.VBUS, SJ402.1
- new net N$4: SJ402.2, U401.CBUS1
- new net PA_AF_DIFF+: R344.2, R345.2, U406.+IN
- new net PA_AF_DIFF-: R346.2, R347.1, U406.-IN
- new net PA_AF_FB: R341.2, R342.1, U405B.-IN
- new net PA_AF_FB_VAR: R342.2, RV303.A
- new net PA_AF_IN: C356.1, R341.1
- new net PA_AF_INT: C357.2, RV303.S, U405B.OUT
- new net PA_AF_INT_COUPLED: C357.1, DN300.AC1, R343.2
- new net PA_AF_OUT: R347.2, R348.1, U406.OUT
- new net PA_AF_RECT+: DN300.DC+, R344.1
- new net PA_AF_RECT-: DN300.DC-, R346.1
- new net PA_AMPLITUDE: C358.1, R348.2, U400.RC5
- new net VBAT_PREFUSE: F100.1, R100.1, XBT100.+
- net 12V: now also J403A.P$1, U405A.V+; no longer U305.V+
- net 3.3V: now also C400.1, C401.1, J400.2, R401.2, R404.1, RV400.E, SJ400.1, U401.3V3OUT, U401.VCC, U401.VCCIO, U406.V+, XDS400.VDD
- net 3.8V: now also A400.BAT_IN
- net 5V: now also SJ400.3, SJ401.1
- net 6V: now also U405A.+IN, U405B.+IN; no longer U305.+IN
- net AMP_!CLIP_OTW: now also U400.RC3
- net AMP_!FAULT: now also U400.RC2
- net AMP_!RESET: now also Q401.D, Q402.D, R404.2
- net AMP_A_FUSED: now also XLS300.+; no longer XLS300.1
- net AMP_B_FILT: now also XLS300.-; no longer XLS300.2
- net AMP_C_FUSED: now also XLS301.+; no longer XLS301.1
- net AMP_D_FUSED: now also XLS302.+; no longer XLS302.1
- net BAT_PRES_SW: now also SW100.2; no longer J100B.P$1
- net BAT_VDD: now also SW100.1; no longer J100A.P$1
- net GND: now also A400.GND, C358.2, C400.2, C401.2, C402.2, C403.2, C404.2, C405.2, C406.2, C407.2, D103.A, D400.C, DN300.AC2, J100.2, J400.3, J401.GND, J402C.P$1, Q400.S, Q401.S, Q402.S, Q403.S, Q404.S, Q405.S, R343.1, R345.1, R402.1, R403.1, R405.1, RV400.A, SJ403.1, SW400C.O, SW400D.O, SW400E.O, SW402.2, SW403.2, SW404.2, SW405.2, SW406.2, SW407.1, SW408.2, SW409.2, U401.GND, U401.GND@1, U405A.V-, U406.V-, XDS400.VSS, XLS301.-, XLS302.-; no longer U305.V-, XLS301.2, XLS302.2
- net PA_B_IN_BUFFERED: now also C356.2, U405A.OUT; no longer U305.OUT
- net PA_B_IN_SUM: now also U405A.-IN; no longer U305.-IN
- net VBAT: now also F100.2; no longer R100.1, XBT100.+
- net VIN_EXT: now also D103.C, J100.1
Other:
- moved on the sheet: A400

Commit message: Finished up digital section, schematic done for now.
Parts:
- added F101: 10A, BW-PassiveMechanical:2410-FUSE
- added J404: SWLED, BW-Connectors:GEN-3PIN
- added Q406, Q407: NMOS, BW-Active:SOT23-N-MOSFET
- D103: value (none) -> SMF28A-M3
Connections:
- net N$1 renamed USB_D+
- net N$2 renamed USB_D-
- net N$3 renamed USB_VBUS
- net N$4 renamed FT_VBUS_SENSE
- new net MCU_SWLED_MAIN: Q406.G, U400.RD6
- new net MCU_SWLED_PWR: Q407.G, U400.RD7
- new net SWLED_MAIN: J404B.P$1, Q406.D
- new net SWLED_PWR: J404C.P$1, Q407.D
- new net VIN_EXT_FUSED: C126.1, C127.1, D100.A, F101.2, Q104.S, U102.ANODE, U102.EN
- net 3.3V: now also U400.VDD
- net 5V: now also J404A.P$1
- net GND: now also Q406.S, Q407.S, U400.VSS
- net LED_G: now also Q403.D; no longer Q404.D
- net LED_R: now also Q404.D; no longer Q403.D
- net MCU_LED_B: now also U400.RD5; no longer U400.RD6
- net MCU_LED_G: now also Q403.G, U400.RC7; no longer Q404.G, U400.RD5
- net MCU_LED_R: now also Q404.G; no longer Q403.G
- net VIN_EXT: now also F101.1; no longer C126.1, C127.1, D100.A, Q104.S, U102.ANODE, U102.EN
Other:
- moved on the sheet: C400, C401, J403A, J403B, J403C, J403D, Q403, Q404, Q405

Commit message: Design initially completed.
Parts:
- removed SW409: LEDSW, BW-PassiveMechanical:WIRED-SWITCH-NO
- added C228: 47µF, rcl:CPOL-EUE2.5-6
- added C409: 0.1µF, rcl:C-EUC0805
- added C410, C411: 0.1µF?, rcl:C-EUC0805
- added J405: USB1, BW-Connectors:GEN-2PIN
- added J406: USB2, BW-Connectors:GEN-2PIN
- added R406: 10kΩ, resistor:R-US_R0805
- added R407: 1.69kΩ, resistor:R-US_R0603
- added R408, R409: 47Ω?, resistor:R-US_R0603
- added RV401: 100kΩ, BW-PassiveMechanical:WIRED-POTENTIOMETER
- added SJ404: GND CUT, jumper:SJ
- added U402: NCS20071, BW-Active:NCS20071
- C308, C309, C315, C321: device rcl:C-EUC0805 -> rcl:C-EUC0603
- C314, C320: value 10µF? -> 10µF
- C334, C335, C337, C338: value 1µF 100V -> 1µF 100V .5
- C341, C342, C344, C345, C347, C348, C350, C351: device rcl:C-EUC1206 -> rcl:C-EUC0603
- FAN300: value HA30101V3 -> 12V <50mA
- J400: value PINHD-1X8 -> ICSP
- Q203: value DMP4065S-7 -> DMP4065S
- R108: value 4.5kΩ -> 4.53kΩ
- SW408: value LCD_BL -> LCDBL
- U203: value MIC5504-3.3YM5-TR -> LDO-3.3V
- U204: value MIC5205-3.8YM5-TR -> LDO-3.8V
- U400: value PIC18LF4_K42-I/PT -> PIC18LF4_K42; device BW-Active:PIC18LF4_K42-I/PT -> BW-Active:PIC18LF4_K42
- XLS300: value SP-6/108PRO -> BASS
- XLS301: value DT-74/8 -> LEFT
- XLS302: value DT74/8 -> RIGHT
- renumbered U405 to U305, U406 to U306
Connections:
- removed net MCU_LED_SW: SW409.1, U400.RC6
- new net BM_SPKL: A400.SPKL, R409.2
- new net BM_SPKR: A400.SPKR, R408.2
- new net MCU_BAT_SENSE: U400.RD3, U402.-IN, U402.OUT
- new net MCU_BAT_VDIV: R406.1, R407.2, U402.+IN
- new net MCU_LED_POT: RV401.S, U400.RC6
- net 12V: now also C228.+
- net 3.3V: now also C409.1, RV401.E, U402.V+
- net 52V: no longer C333.1
- net 5V: now also J405A.P$1, J406A.P$1
- net AMP_OUT_D: now also C333.1
- net AUD_SRC_L: now also C411.1, R409.1; no longer A400.SPKL
- net AUD_SRC_R: now also C410.2, R408.1; no longer A400.SPKR
- net BUCK_FB: now also C226.2
- net FT_RXD: now also SW400B.O; no longer SW400B.S
- net FT_TXD: now also SW400A.O; no longer SW400A.S
- net GND: now also C228.-, C409.2, C410.1, C411.2, J405B.P$1, J406B.P$1, R407.1, RV401.A, SJ404.1, SJ404.2, SW400C.S, SW400D.S, SW400E.S, U402.V-; no longer C226.2, SW400C.O, SW400D.O, SW400E.O, SW409.2
- net MCU_UART_RX: now also SW400B.S; no longer SW400B.O
- net MCU_UART_TX: now also SW400A.S; no longer SW400A.O
- net VBAT: now also R406.2
Other:
- note added: "Shortcut between digital and low-power analog ground planes in case of issues"

Commit message: Final checks and fixes applied.
Other:
- moved on the sheet: C335, C336, C337, C338, C339
Changed lines of the file:
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@@
 <attribute name="VALUE" x="-49.657" y="-7.1374" size="1.778" layer="96"/>
 </instance>
-<instance part="C336" gate="G$1" x="124.46" y="-12.7" smashed="yes">
-<attribute name="NAME" x="125.603" y="-12.2174" size="1.778" layer="95"/>
-<attribute name="VALUE" x="125.603" y="-17.2974" size="1.778" layer="96"/>
+<instance part="C336" gate="G$1" x="129.54" y="-12.7" smashed="yes">
+<attribute name="NAME" x="130.683" y="-12.2174" size="1.778" layer="95"/>
+<attribute name="VALUE" x="130.683" y="-17.2974" size="1.778" layer="96"/>
 </instance>
 <instance part="C323" gate="G$1" x="-40.64" y="-2.54" smashed="yes">
@@
 <attribute name="VALUE" x="-39.116" y="-7.239" size="1.778" layer="96"/>
 </instance>
-<instance part="C339" gate="G$1" x="165.1" y="-12.7" smashed="yes">
-<attribute name="NAME" x="166.243" y="-12.2174" size="1.778" layer="95"/>
-<attribute name="VALUE" x="166.243" y="-17.2974" size="1.778" layer="96"/>
+<instance part="C339" gate="G$1" x="175.26" y="-12.7" smashed="yes">
+<attribute name="NAME" x="176.403" y="-12.2174" size="1.778" layer="95"/>
+<attribute name="VALUE" x="176.403" y="-17.2974" size="1.778" layer="96"/>
 </instance>
 <instance part="C324" gate="G$1" x="-22.86" y="-2.54" smashed="yes">
@@
 <attribute name="VALUE" x="21.844" y="-7.239" size="1.778" layer="96"/>
 </instance>
-<instance part="C337" gate="G$1" x="139.7" y="-12.7" smashed="yes">
-<attribute name="NAME" x="141.224" y="-12.319" size="1.778" layer="95"/>
-<attribute name="VALUE" x="141.224" y="-17.399" size="1.778" layer="96"/>
-</instance>
-<instance part="C338" gate="G$1" x="152.4" y="-12.7" smashed="yes">
-<attribute name="NAME" x="153.924" y="-12.319" size="1.778" layer="95"/>
-<attribute name="VALUE" x="153.924" y="-17.399" size="1.778" layer="96"/>
-</instance>
-<instance part="C335" gate="G$1" x="111.76" y="-12.7" smashed="yes">
-<attribute name="NAME" x="113.284" y="-12.319" size="1.778" layer="95"/>
-<attribute name="VALUE" x="113.284" y="-17.399" size="1.778" layer="96"/>
+<instance part="C337" gate="G$1" x="144.78" y="-12.7" smashed="yes">
+<attribute name="NAME" x="146.304" y="-12.319" size="1.778" layer="95"/>
+<attribute name="VALUE" x="146.304" y="-17.399" size="1.778" layer="96"/>
+</instance>
+<instance part="C338" gate="G$1" x="160.02" y="-12.7" smashed="yes">
+<attribute name="NAME" x="161.544" y="-12.319" size="1.778" layer="95"/>
+<attribute name="VALUE" x="161.544" y="-17.399" size="1.778" layer="96"/>
+</instance>
+<instance part="C335" gate="G$1" x="114.3" y="-12.7" smashed="yes">
+<attribute name="NAME" x="115.824" y="-12.319" size="1.778" layer="95"/>
+<attribute name="VALUE" x="115.824" y="-17.399" size="1.778" layer="96"/>
 </instance>
 <instance part="C334" gate="G$1" x="99.06" y="-12.7" smashed="yes">
@@
 <pinref part="C334" gate="G$1" pin="2"/>
 <wire x1="99.06" y1="-17.78" x2="99.06" y2="-20.32" width="0.1524" layer="91"/>
-<wire x1="99.06" y1="-20.32" x2="111.76" y2="-20.32" width="0.1524" layer="91"/>
+<wire x1="99.06" y1="-20.32" x2="114.3" y2="-20.32" width="0.1524" layer="91"/>
 <pinref part="C339" gate="G$1" pin="-"/>
-<wire x1="111.76" y1="-20.32" x2="124.46" y2="-20.32" width="0.1524" layer="91"/>
-<wire x1="124.46" y1="-20.32" x2="132.08" y2="-20.32" width="0.1524" layer="91"/>
-<wire x1="132.08" y1="-20.32" x2="139.7" y2="-20.32" width="0.1524" layer="91"/>
-<wire x1="139.7" y1="-20.32" x2="152.4" y2="-20.32" width="0.1524" layer="91"/>
-<wire x1="152.4" y1="-20.32" x2="165.1" y2="-20.32" width="0.1524" layer="91"/>
-<wire x1="165.1" y1="-20.32" x2="165.1" y2="-17.78" width="0.1524" layer="91"/>
+<wire x1="114.3" y1="-20.32" x2="129.54" y2="-20.32" width="0.1524" layer="91"/>
+<wire x1="129.54" y1="-20.32" x2="137.16" y2="-20.32" width="0.1524" layer="91"/>
+<wire x1="137.16" y1="-20.32" x2="144.78" y2="-20.32" width="0.1524" layer="91"/>
+<wire x1="144.78" y1="-20.32" x2="160.02" y2="-20.32" width="0.1524" layer="91"/>
+<wire x1="160.02" y1="-20.32" x2="175.26" y2="-20.32" width="0.1524" layer="91"/>
+<wire x1="175.26" y1="-20.32" x2="175.26" y2="-17.78" width="0.1524" layer="91"/>
 <pinref part="C335" gate="G$1" pin="2"/>
-<wire x1="111.76" y1="-17.78" x2="111.76" y2="-20.32" width="0.1524" layer="91"/>
-<junction x="111.76" y="-20.32"/>
+<wire x1="114.3" y1="-17.78" x2="114.3" y2="-20.32" width="0.1524" layer="91"/>
+<junction x="114.3" y="-20.32"/>
 <pinref part="C336" gate="G$1" pin="-"/>
-<wire x1="124.46" y1="-17.78" x2="124.46" y2="-20.32" width="0.1524" layer="91"/>
-<junction x="124.46" y="-20.32"/>
+<wire x1="129.54" y1="-17.78" x2="129.54" y2="-20.32" width="0.1524" layer="91"/>
+<junction x="129.54" y="-20.32"/>
 <pinref part="C337" gate="G$1" pin="2"/>
-<wire x1="139.7" y1="-17.78" x2="139.7" y2="-20.32" width="0.1524" layer="91"/>
-<junction x="139.7" y="-20.32"/>
+<wire x1="144.78" y1="-17.78" x2="144.78" y2="-20.32" width="0.1524" layer="91"/>
+<junction x="144.78" y="-20.32"/>
 <pinref part="C338" gate="G$1" pin="2"/>
-<wire x1="152.4" y1="-17.78" x2="152.4" y2="-20.32" width="0.1524" layer="91"/>
-<junction x="152.4" y="-20.32"/>
-<wire x1="132.08" y1="-20.32" x2="132.08" y2="-22.86" width="0.1524" layer="91"/>
-<junction x="132.08" y="-20.32"/>
-<label x="132.08" y="-25.4" size="1.778" layer="95"/>
+<wire x1="160.02" y1="-17.78" x2="160.02" y2="-20.32" width="0.1524" layer="91"/>
+<junction x="160.02" y="-20.32"/>
+<wire x1="137.16" y1="-20.32" x2="137.16" y2="-22.86" width="0.1524" layer="91"/>
+<junction x="137.16" y="-20.32"/>
+<label x="137.16" y="-25.4" size="1.778" layer="95"/>
 </segment>
 <segment>
@@
 <junction x="99.06" y="-7.62"/>
 <pinref part="C335" gate="G$1" pin="1"/>
-<wire x1="111.76" y1="-7.62" x2="99.06" y2="-7.62" width="0.1524" layer="91"/>
-<wire x1="111.76" y1="-10.16" x2="111.76" y2="-7.62" width="0.1524" layer="91"/>
+<wire x1="114.3" y1="-7.62" x2="99.06" y2="-7.62" width="0.1524" layer="91"/>
+<wire x1="114.3" y1="-10.16" x2="114.3" y2="-7.62" width="0.1524" layer="91"/>
 <pinref part="C336" gate="G$1" pin="+"/>
-<wire x1="124.46" y1="-10.16" x2="124.46" y2="-7.62" width="0.1524" layer="91"/>
-<wire x1="124.46" y1="-7.62" x2="111.76" y2="-7.62" width="0.1524" layer="91"/>
-<junction x="111.76" y="-7.62"/>
+<wire x1="129.54" y1="-10.16" x2="129.54" y2="-7.62" width="0.1524" layer="91"/>
+<wire x1="129.54" y1="-7.62" x2="114.3" y2="-7.62" width="0.1524" layer="91"/>
+<junction x="114.3" y="-7.62"/>
 <pinref part="C337" gate="G$1" pin="1"/>
 <pinref part="C339" gate="G$1" pin="+"/>
-<wire x1="165.1" y1="-10.16" x2="165.1" y2="-7.62" width="0.1524" layer="91"/>
-<wire x1="165.1" y1="-7.62" x2="152.4" y2="-7.62" width="0.1524" layer="91"/>
+<wire x1="175.26" y1="-10.16" x2="175.26" y2="-7.62" width="0.1524" layer="91"/>
+<wire x1="175.26" y1="-7.62" x2="160.02" y2="-7.62" width="0.1524" layer="91"/>
 <pinref part="C338" gate="G$1" pin="1"/>
-<wire x1="152.4" y1="-10.16" x2="152.4" y2="-7.62" width="0.1524" layer="91"/>
-<junction x="152.4" y="-7.62"/>
-<wire x1="152.4" y1="-7.62" x2="139.7" y2="-7.62" width="0.1524" layer="91"/>
-<wire x1="139.7" y1="-7.62" x2="139.7" y2="-10.16" width="0.1524" layer="91"/>
-<wire x1="124.46" y1="-7.62" x2="139.7" y2="-7.62" width="0.1524" layer="91"/>
-<junction x="124.46" y="-7.62"/>
-<junction x="139.7" y="-7.62"/>
+<wire x1="160.02" y1="-10.16" x2="160.02" y2="-7.62" width="0.1524" layer="91"/>
+<junction x="160.02" y="-7.62"/>
+<wire x1="160.02" y1="-7.62" x2="144.78" y2="-7.62" width="0.1524" layer="91"/>
+<wire x1="144.78" y1="-7.62" x2="144.78" y2="-10.16" width="0.1524" layer="91"/>
+<wire x1="129.54" y1="-7.62" x2="144.78" y2="-7.62" width="0.1524" layer="91"/>
+<junction x="129.54" y="-7.62"/>
+<junction x="144.78" y="-7.62"/>
 <pinref part="U300" gate="G$1" pin="PVDD_AB"/>
 <wire x1="99.06" y1="20.32" x2="99.06" y2="38.1" width="0.1524" layer="91"/>
