File: ButtonBoard.sch (EAGLE design)
At the start: 23 parts, among them J1 MFB, J2 VOL-, J3 VOL+, J4 BACK, J5 PLAY, J6 FWD, J7 LED, SW1 TC012A, SW2 TC012A, SW3 TC012A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

Commit message: Final checks and fixes applied.
Parts:
- J1: value MFB -> VOL-
- J2: value VOL- -> MFB
Connections:
- net LED_MAIN_5: now also R1.2; no longer R2.2
- net LED_MAIN_6: now also SW1L.C; no longer SW2L.C
- net LED_MFB_5: now also R2.2; no longer R1.2
- net LED_MFB_5R: now also R2.1, SW2L.A; no longer R1.1, SW1L.A
- net LED_MFB_6: now also SW2L.C; no longer SW1L.C
- net LED_VOL-_5R: now also R1.1, SW1L.A; no longer R2.1, SW2L.A
- net MFB1: now also J2A.P$1, SW2S.1; no longer J1A.P$1, SW1S.1
- net MFB2: now also J2B.P$1, SW2S.2; no longer J1B.P$1, SW1S.2
- net VOL-1: now also J1A.P$1, SW1S.1; no longer J2A.P$1, SW2S.1
- net VOL-2: now also J1B.P$1, SW1S.2; no longer J2B.P$1, SW2S.2
Other:
- moved on the sheet: R1, R2, SW1L, SW2L
Changed lines of the file:
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@@
 <part name="SW5" library="BW-PassiveMechanical" deviceset="TC012A" device=""/>
 <part name="SW6" library="BW-PassiveMechanical" deviceset="TC012A" device=""/>
-<part name="J1" library="BW-Connectors" deviceset="GEN-2PIN" device="" value="MFB"/>
-<part name="J2" library="BW-Connectors" deviceset="GEN-2PIN" device="" value="VOL-"/>
+<part name="J1" library="BW-Connectors" deviceset="GEN-2PIN" device="" value="VOL-"/>
+<part name="J2" library="BW-Connectors" deviceset="GEN-2PIN" device="" value="MFB"/>
 <part name="J3" library="BW-Connectors" deviceset="GEN-2PIN" device="" value="VOL+"/>
 <part name="J4" library="BW-Connectors" deviceset="GEN-2PIN" device="" value="BACK"/>
@@
 <attribute name="VALUE" x="-21.59" y="46.99" size="1.778" layer="96"/>
 </instance>
-<instance part="SW1" gate="L" x="-27.94" y="-33.02" smashed="yes">
-<attribute name="NAME" x="-24.384" y="-37.592" size="1.778" layer="95" rot="R90"/>
-<attribute name="VALUE" x="-22.225" y="-37.592" size="1.778" layer="96" rot="R90"/>
+<instance part="SW1" gate="L" x="-7.62" y="-33.02" smashed="yes">
+<attribute name="NAME" x="-4.064" y="-37.592" size="1.778" layer="95" rot="R90"/>
+<attribute name="VALUE" x="-1.905" y="-37.592" size="1.778" layer="96" rot="R90"/>
 </instance>
 <instance part="SW2" gate="S" x="5.08" y="50.8" smashed="yes">
@@
 <attribute name="VALUE" x="1.27" y="46.99" size="1.778" layer="96"/>
 </instance>
-<instance part="SW2" gate="L" x="-7.62" y="-33.02" smashed="yes">
-<attribute name="NAME" x="-4.064" y="-37.592" size="1.778" layer="95" rot="R90"/>
-<attribute name="VALUE" x="-1.905" y="-37.592" size="1.778" layer="96" rot="R90"/>
+<instance part="SW2" gate="L" x="-27.94" y="-33.02" smashed="yes">
+<attribute name="NAME" x="-24.384" y="-37.592" size="1.778" layer="95" rot="R90"/>
+<attribute name="VALUE" x="-22.225" y="-37.592" size="1.778" layer="96" rot="R90"/>
 </instance>
 <instance part="SW3" gate="S" x="27.94" y="50.8" smashed="yes">
@@
 <attribute name="VALUE" x="-53.34" y="-23.876" size="1.27" layer="96" rot="R180"/>
 </instance>
-<instance part="R1" gate="G$1" x="-27.94" y="-20.32" smashed="yes" rot="R90">
+<instance part="R1" gate="G$1" x="-7.62" y="-20.32" smashed="yes" rot="R90">
+<attribute name="NAME" x="-9.1186" y="-24.13" size="1.778" layer="95" rot="R90"/>
+<attribute name="VALUE" x="-4.318" y="-24.13" size="1.778" layer="96" rot="R90"/>
+</instance>
+<instance part="R2" gate="G$1" x="-27.94" y="-20.32" smashed="yes" rot="R90">
 <attribute name="NAME" x="-29.4386" y="-24.13" size="1.778" layer="95" rot="R90"/>
 <attribute name="VALUE" x="-24.638" y="-24.13" size="1.778" layer="96" rot="R90"/>
-</instance>
-<instance part="R2" gate="G$1" x="-7.62" y="-20.32" smashed="yes" rot="R90">
-<attribute name="NAME" x="-9.1186" y="-24.13" size="1.778" layer="95" rot="R90"/>
-<attribute name="VALUE" x="-4.318" y="-24.13" size="1.778" layer="96" rot="R90"/>
 </instance>
 <instance part="R3" gate="G$1" x="7.62" y="-20.32" smashed="yes" rot="R90">
@@
 </busses>
 <nets>
-<net name="MFB1" class="0">
+<net name="VOL-1" class="0">
 <segment>
 <pinref part="J1" gate="A" pin="P$1"/>
@@
 </segment>
 </net>
-<net name="MFB2" class="0">
+<net name="VOL-2" class="0">
 <segment>
 <pinref part="J1" gate="B" pin="P$1"/>
@@
 </segment>
 </net>
-<net name="VOL-1" class="0">
+<net name="MFB1" class="0">
 <segment>
 <pinref part="J2" gate="A" pin="P$1"/>
@@
 </segment>
 </net>
-<net name="VOL-2" class="0">
+<net name="MFB2" class="0">
 <segment>
 <pinref part="J2" gate="B" pin="P$1"/>
@@
 <pinref part="SJ1" gate="G$1" pin="2"/>
 <wire x1="-33.02" y1="-12.7" x2="-27.94" y2="-12.7" width="0.1524" layer="91"/>
-<pinref part="R1" gate="G$1" pin="2"/>
+<pinref part="R2" gate="G$1" pin="2"/>
 <wire x1="-27.94" y1="-15.24" x2="-27.94" y2="-12.7" width="0.1524" layer="91"/>
 </segment>
@@
 <segment>
 <pinref part="SJ2" gate="G$1" pin="2"/>
-<pinref part="SW1" gate="L" pin="C"/>
 <wire x1="-33.02" y1="-40.64" x2="-27.94" y2="-40.64" width="0.1524" layer="91"/>
-<wire x1="-27.94" y1="-40.64" x2="-27.94" y2="-38.1" width="0.1524" layer="91"/>
+<pinref part="SW2" gate="L" pin="C"/>
+<wire x1="-27.94" y1="-38.1" x2="-27.94" y2="-40.64" width="0.1524" layer="91"/>
 </segment>
 </net>
@@
 <pinref part="SJ3" gate="G$1" pin="2"/>
 <wire x1="60.96" y1="-12.7" x2="53.34" y2="-12.7" width="0.1524" layer="91"/>
-<pinref part="R2" gate="G$1" pin="2"/>
 <wire x1="53.34" y1="-12.7" x2="38.1" y2="-12.7" width="0.1524" layer="91"/>
 <wire x1="38.1" y1="-12.7" x2="22.86" y2="-12.7" width="0.1524" layer="91"/>
 <wire x1="22.86" y1="-12.7" x2="7.62" y2="-12.7" width="0.1524" layer="91"/>
 <wire x1="7.62" y1="-12.7" x2="-7.62" y2="-12.7" width="0.1524" layer="91"/>
-<wire x1="-7.62" y1="-15.24" x2="-7.62" y2="-12.7" width="0.1524" layer="91"/>
 <pinref part="R6" gate="G$1" pin="2"/>
 <wire x1="53.34" y1="-15.24" x2="53.34" y2="-12.7" width="0.1524" layer="91"/>
@@
 <wire x1="7.62" y1="-15.24" x2="7.62" y2="-12.7" width="0.1524" layer="91"/>
 <junction x="7.62" y="-12.7"/>
+<pinref part="R1" gate="G$1" pin="2"/>
+<wire x1="-7.62" y1="-15.24" x2="-7.62" y2="-12.7" width="0.1524" layer="91"/>
 </segment>
 </net>
 <net name="LED_MAIN_6" class="0">
 <segment>
-<pinref part="SW2" gate="L" pin="C"/>
 <pinref part="SJ4" gate="G$1" pin="2"/>
-<wire x1="-7.62" y1="-38.1" x2="-7.62" y2="-40.64" width="0.1524" layer="91"/>
 <wire x1="-7.62" y1="-40.64" x2="7.62" y2="-40.64" width="0.1524" layer="91"/>
 <pinref part="SW3" gate="L" pin="C"/>
@@
 <wire x1="53.34" y1="-38.1" x2="53.34" y2="-40.64" width="0.1524" layer="91"/>
 <junction x="53.34" y="-40.64"/>
+<pinref part="SW1" gate="L" pin="C"/>
+<wire x1="-7.62" y1="-38.1" x2="-7.62" y2="-40.64" width="0.1524" layer="91"/>
 </segment>
 </net>
@@
 </segment>
 </net>
-<net name="LED_MFB_5R" class="0">
+<net name="LED_VOL-_5R" class="0">
 <segment>
 <pinref part="R1" gate="G$1" pin="1"/>
 <pinref part="SW1" gate="L" pin="A"/>
-<wire x1="-27.94" y1="-25.4" x2="-27.94" y2="-30.48" width="0.1524" layer="91"/>
-</segment>
-</net>
-<net name="LED_VOL-_5R" class="0">
+<wire x1="-7.62" y1="-25.4" x2="-7.62" y2="-30.48" width="0.1524" layer="91"/>
+</segment>
+</net>
+<net name="LED_MFB_5R" class="0">
 <segment>
 <pinref part="R2" gate="G$1" pin="1"/>
 <pinref part="SW2" gate="L" pin="A"/>
-<wire x1="-7.62" y1="-25.4" x2="-7.62" y2="-30.48" width="0.1524" layer="91"/>
-</segment>
-</net>
+<wire x1="-27.94" y1="-25.4" x2="-27.94" y2="-30.48" width="0.1524" layer="91"/>
+</segment>
+</net>
